File: hardware/kicad/boosta/boosta.kicad_pcb (KiCad board)
At the start: 2 copper layers, 100.9 x 90.4 mm, 2 parts, among them J1 Conn_01x08_Female, J2 Screw_Terminal_01x02

Commit message: update
Parts:
- moved J1 17.8 mm to (91.5, 55.4), turned to 0 degrees
Changed lines of the file:
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@@
       (effects (font (size 1 1) (thickness 0.15)))
     )
+    (fp_line (start 8.13 -5.71) (end -3.04 -5.71) (layer F.CrtYd) (width 0.05))
+    (fp_line (start 8.13 5.1) (end 8.13 -5.71) (layer F.CrtYd) (width 0.05))
+    (fp_line (start -3.04 5.1) (end 8.13 5.1) (layer F.CrtYd) (width 0.05))
+    (fp_line (start -3.04 -5.71) (end -3.04 5.1) (layer F.CrtYd) (width 0.05))
+    (fp_line (start -2.84 4.9) (end -2.34 4.9) (layer F.SilkS) (width 0.12))
+    (fp_line (start -2.84 4.16) (end -2.84 4.9) (layer F.SilkS) (width 0.12))
+    (fp_line (start 3.853 1.023) (end 3.806 1.069) (layer F.SilkS) (width 0.12))
+    (fp_line (start 6.15 -1.275) (end 6.115 -1.239) (layer F.SilkS) (width 0.12))
+    (fp_line (start 4.046 1.239) (end 4.011 1.274) (layer F.SilkS) (width 0.12))
+    (fp_line (start 6.355 -1.069) (end 6.308 -1.023) (layer F.SilkS) (width 0.12))
+    (fp_line (start 6.035 -1.138) (end 3.943 0.955) (layer F.Fab) (width 0.1))
+    (fp_line (start 6.218 -0.955) (end 4.126 1.138) (layer F.Fab) (width 0.1))
+    (fp_line (start 0.955 -1.138) (end -1.138 0.955) (layer F.Fab) (width 0.1))
+    (fp_line (start 1.138 -0.955) (end -0.955 1.138) (layer F.Fab) (width 0.1))
+    (fp_line (start 7.68 -5.261) (end 7.68 4.66) (layer F.SilkS) (width 0.12))
+    (fp_line (start -2.6 -5.261) (end -2.6 4.66) (layer F.SilkS) (width 0.12))
+    (fp_line (start -2.6 4.66) (end 7.68 4.66) (layer F.SilkS) (width 0.12))
+    (fp_line (start -2.6 -5.261) (end 7.68 -5.261) (layer F.SilkS) (width 0.12))
+    (fp_line (start -2.6 -2.301) (end 7.68 -2.301) (layer F.SilkS) (width 0.12))
+    (fp_line (start -2.54 -2.3) (end 7.62 -2.3) (layer F.Fab) (width 0.1))
+    (fp_line (start -2.6 2.6) (end 7.68 2.6) (layer F.SilkS) (width 0.12))
+    (fp_line (start -2.54 2.6) (end 7.62 2.6) (layer F.Fab) (width 0.1))
+    (fp_line (start -2.6 4.1) (end 7.68 4.1) (layer F.SilkS) (width 0.12))
+    (fp_line (start -2.54 4.1) (end 7.62 4.1) (layer F.Fab) (width 0.1))
+    (fp_line (start -2.54 4.1) (end -2.54 -5.2) (layer F.Fab) (width 0.1))
+    (fp_line (start -2.04 4.6) (end -2.54 4.1) (layer F.Fab) (width 0.1))
+    (fp_line (start 7.62 4.6) (end -2.04 4.6) (layer F.Fab) (width 0.1))
+    (fp_line (start 7.62 -5.2) (end 7.62 4.6) (layer F.Fab) (width 0.1))
+    (fp_line (start -2.54 -5.2) (end 7.62 -5.2) (layer F.Fab) (width 0.1))
+    (fp_circle (center 5.08 0) (end 6.76 0) (layer F.SilkS) (width 0.12))
+    (fp_circle (center 5.08 0) (end 6.58 0) (layer F.Fab) (width 0.1))
+    (fp_circle (center 0 0) (end 1.5 0) (layer F.Fab) (width 0.1))
     (fp_text user %R (at 2.54 3.2 90) (layer F.Fab)
       (effects (font (size 1 1) (thickness 0.15)))
@@
     (fp_arc (start 0 0) (end 1.535 0.684) (angle -48) (layer F.SilkS) (width 0.12))
     (fp_arc (start 0 0) (end 0 1.68) (angle -24) (layer F.SilkS) (width 0.12))
-    (fp_circle (center 0 0) (end 1.5 0) (layer F.Fab) (width 0.1))
-    (fp_circle (center 5.08 0) (end 6.58 0) (layer F.Fab) (width 0.1))
-    (fp_circle (center 5.08 0) (end 6.76 0) (layer F.SilkS) (width 0.12))
-    (fp_line (start -2.54 -5.2) (end 7.62 -5.2) (layer F.Fab) (width 0.1))
-    (fp_line (start 7.62 -5.2) (end 7.62 4.6) (layer F.Fab) (width 0.1))
-    (fp_line (start 7.62 4.6) (end -2.04 4.6) (layer F.Fab) (width 0.1))
-    (fp_line (start -2.04 4.6) (end -2.54 4.1) (layer F.Fab) (width 0.1))
-    (fp_line (start -2.54 4.1) (end -2.54 -5.2) (layer F.Fab) (width 0.1))
-    (fp_line (start -2.54 4.1) (end 7.62 4.1) (layer F.Fab) (width 0.1))
-    (fp_line (start -2.6 4.1) (end 7.68 4.1) (layer F.SilkS) (width 0.12))
-    (fp_line (start -2.54 2.6) (end 7.62 2.6) (layer F.Fab) (width 0.1))
-    (fp_line (start -2.6 2.6) (end 7.68 2.6) (layer F.SilkS) (width 0.12))
-    (fp_line (start -2.54 -2.3) (end 7.62 -2.3) (layer F.Fab) (width 0.1))
-    (fp_line (start -2.6 -2.301) (end 7.68 -2.301) (layer F.SilkS) (width 0.12))
-    (fp_line (start -2.6 -5.261) (end 7.68 -5.261) (layer F.SilkS) (width 0.12))
-    (fp_line (start -2.6 4.66) (end 7.68 4.66) (layer F.SilkS) (width 0.12))
-    (fp_line (start -2.6 -5.261) (end -2.6 4.66) (layer F.SilkS) (width 0.12))
-    (fp_line (start 7.68 -5.261) (end 7.68 4.66) (layer F.SilkS) (width 0.12))
-    (fp_line (start 1.138 -0.955) (end -0.955 1.138) (layer F.Fab) (width 0.1))
-    (fp_line (start 0.955 -1.138) (end -1.138 0.955) (layer F.Fab) (width 0.1))
-    (fp_line (start 6.218 -0.955) (end 4.126 1.138) (layer F.Fab) (width 0.1))
-    (fp_line (start 6.035 -1.138) (end 3.943 0.955) (layer F.Fab) (width 0.1))
-    (fp_line (start 6.355 -1.069) (end 6.308 -1.023) (layer F.SilkS) (width 0.12))
-    (fp_line (start 4.046 1.239) (end 4.011 1.274) (layer F.SilkS) (width 0.12))
-    (fp_line (start 6.15 -1.275) (end 6.115 -1.239) (layer F.SilkS) (width 0.12))
-    (fp_line (start 3.853 1.023) (end 3.806 1.069) (layer F.SilkS) (width 0.12))
-    (fp_line (start -2.84 4.16) (end -2.84 4.9) (layer F.SilkS) (width 0.12))
-    (fp_line (start -2.84 4.9) (end -2.34 4.9) (layer F.SilkS) (width 0.12))
-    (fp_line (start -3.04 -5.71) (end -3.04 5.1) (layer F.CrtYd) (width 0.05))
-    (fp_line (start -3.04 5.1) (end 8.13 5.1) (layer F.CrtYd) (width 0.05))
-    (fp_line (start 8.13 5.1) (end 8.13 -5.71) (layer F.CrtYd) (width 0.05))
-    (fp_line (start 8.13 -5.71) (end -3.04 -5.71) (layer F.CrtYd) (width 0.05))
     (pad 2 thru_hole circle (at 5.08 0 270) (size 2.6 2.6) (drill 1.3) (layers *.Cu *.Mask)
       (net 2 5V))
@@
   )
   (module Connector_PinSocket_2.54mm:PinSocket_1x08_P2.54mm_Vertical (layer F.Cu)
-    (at 91.35 73.15 180)
+    (at 91.55 55.35)
     (descr "Through hole straight socket strip, 1x08, 2.54mm pitch, single row (from Kicad 4.0.7), script generated")
     (tags "Through hole socket strip THT 1x08 2.54mm single row")
@@
       (effects (font (size 1 1) (thickness 0.15)))
     )
+    (fp_line (start -1.8 19.55) (end -1.8 -1.8) (layer F.CrtYd) (width 0.05))
+    (fp_line (start 1.75 19.55) (end -1.8 19.55) (layer F.CrtYd) (width 0.05))
+    (fp_line (start 1.75 -1.8) (end 1.75 19.55) (layer F.CrtYd) (width 0.05))
+    (fp_line (start -1.8 -1.8) (end 1.75 -1.8) (layer F.CrtYd) (width 0.05))
+    (fp_line (start 0 -1.33) (end 1.33 -1.33) (layer F.SilkS) (width 0.12))
+    (fp_line (start 1.33 -1.33) (end 1.33 0) (layer F.SilkS) (width 0.12))
+    (fp_line (start 1.33 1.27) (end 1.33 19.11) (layer F.SilkS) (width 0.12))
+    (fp_line (start -1.33 19.11) (end 1.33 19.11) (layer F.SilkS) (width 0.12))
+    (fp_line (start -1.33 1.27) (end -1.33 19.11) (layer F.SilkS) (width 0.12))
+    (fp_line (start -1.33 1.27) (end 1.33 1.27) (layer F.SilkS) (width 0.12))
+    (fp_line (start -1.27 19.05) (end -1.27 -1.27) (layer F.Fab) (width 0.1))
+    (fp_line (start 1.27 19.05) (end -1.27 19.05) (layer F.Fab) (width 0.1))
+    (fp_line (start 1.27 -0.635) (end 1.27 19.05) (layer F.Fab) (width 0.1))
+    (fp_line (start 0.635 -1.27) (end 1.27 -0.635) (layer F.Fab) (width 0.1))
+    (fp_line (start -1.27 -1.27) (end 0.635 -1.27) (layer F.Fab) (width 0.1))
     (fp_text user %R (at 0 8.89 90) (layer F.Fab)
       (effects (font (size 1 1) (thickness 0.15)))
     )
-    (fp_line (start -1.27 -1.27) (end 0.635 -1.27) (layer F.Fab) (width 0.1))
-    (fp_line (start 0.635 -1.27) (end 1.27 -0.635) (layer F.Fab) (width 0.1))
-    (fp_line (start 1.27 -0.635) (end 1.27 19.05) (layer F.Fab) (width 0.1))
-    (fp_line (start 1.27 19.05) (end -1.27 19.05) (layer F.Fab) (width 0.1))
-    (fp_line (start -1.27 19.05) (end -1.27 -1.27) (layer F.Fab) (width 0.1))
-    (fp_line (start -1.33 1.27) (end 1.33 1.27) (layer F.SilkS) (width 0.12))
-    (fp_line (start -1.33 1.27) (end -1.33 19.11) (layer F.SilkS) (width 0.12))
-    (fp_line (start -1.33 19.11) (end 1.33 19.11) (layer F.SilkS) (width 0.12))
-    (fp_line (start 1.33 1.27) (end 1.33 19.11) (layer F.SilkS) (width 0.12))
-    (fp_line (start 1.33 -1.33) (end 1.33 0) (layer F.SilkS) (width 0.12))
-    (fp_line (start 0 -1.33) (end 1.33 -1.33) (layer F.SilkS) (width 0.12))
-    (fp_line (start -1.8 -1.8) (end 1.75 -1.8) (layer F.CrtYd) (width 0.05))
-    (fp_line (start 1.75 -1.8) (end 1.75 19.55) (layer F.CrtYd) (width 0.05))
-    (fp_line (start 1.75 19.55) (end -1.8 19.55) (layer F.CrtYd) (width 0.05))
-    (fp_line (start -1.8 19.55) (end -1.8 -1.8) (layer F.CrtYd) (width 0.05))
-    (pad 8 thru_hole oval (at 0 17.78 180) (size 1.7 1.7) (drill 1) (layers *.Cu *.Mask))
-    (pad 7 thru_hole oval (at 0 15.24 180) (size 1.7 1.7) (drill 1) (layers *.Cu *.Mask)
+    (pad 8 thru_hole oval (at 0 17.78) (size 1.7 1.7) (drill 1) (layers *.Cu *.Mask))
+    (pad 7 thru_hole oval (at 0 15.24) (size 1.7 1.7) (drill 1) (layers *.Cu *.Mask)
       (net 1 GND))
-    (pad 6 thru_hole oval (at 0 12.7 180) (size 1.7 1.7) (drill 1) (layers *.Cu *.Mask))
-    (pad 5 thru_hole oval (at 0 10.16 180) (size 1.7 1.7) (drill 1) (layers *.Cu *.Mask))
-    (pad 4 thru_hole oval (at 0 7.62 180) (size 1.7 1.7) (drill 1) (layers *.Cu *.Mask)
+    (pad 6 thru_hole oval (at 0 12.7) (size 1.7 1.7) (drill 1) (layers *.Cu *.Mask))
+    (pad 5 thru_hole oval (at 0 10.16) (size 1.7 1.7) (drill 1) (layers *.Cu *.Mask))
+    (pad 4 thru_hole oval (at 0 7.62) (size 1.7 1.7) (drill 1) (layers *.Cu *.Mask)
       (net 1 GND))
-    (pad 3 thru_hole oval (at 0 5.08 180) (size 1.7 1.7) (drill 1) (layers *.Cu *.Mask))
-    (pad 2 thru_hole oval (at 0 2.54 180) (size 1.7 1.7) (drill 1) (layers *.Cu *.Mask)
+    (pad 3 thru_hole oval (at 0 5.08) (size 1.7 1.7) (drill 1) (layers *.Cu *.Mask))
+    (pad 2 thru_hole oval (at 0 2.54) (size 1.7 1.7) (drill 1) (layers *.Cu *.Mask)
       (net 1 GND))
-    (pad 1 thru_hole rect (at 0 0 180) (size 1.7 1.7) (drill 1) (layers *.Cu *.Mask)
+    (pad 1 thru_hole rect (at 0 0) (size 1.7 1.7) (drill 1) (layers *.Cu *.Mask)
       (net 2 5V))
     (model ${KISYS3DMOD}/Connector_PinSocket_2.54mm.3dshapes/PinSocket_1x08_P2.54mm_Vertical.wrl

Commit message: update
Parts:
- added BT1: Battery_Cell, Battery:BatteryHolder_Keystone_1042_1x18650, F.Cu at (76.5, 105.5)
- added C1: 10uF, Capacitor_THT:CP_Radial_D5.0mm_P2.50mm, F.Cu at (90.0, 130.2)
- added C2: 22uF, Capacitor_THT:CP_Radial_D5.0mm_P2.50mm, F.Cu at (90.0, 123.1)
- added D1: D, Diode_THT:D_5W_P12.70mm_Horizontal, F.Cu at (92.7, 138.0)
- added F1: Polyfuse, Fuse:Fuse_Bourns_MF-RHT1100, F.Cu at (113.2, 140.6)
- added H1: MountingHole_Pad, MountingHole:MountingHole_6.4mm_M6_Pad_Via, F.Cu at (38.4, 85.6)
- added H2: MountingHole_Pad, MountingHole:MountingHole_6.4mm_M6_Pad_Via, F.Cu at (114.5, 85.6)
- added H3: MountingHole, MountingHole:MountingHole_6.4mm_M6, F.Cu at (37.1, 158.8)
- added H4: MountingHole, MountingHole:MountingHole_6.4mm_M6, F.Cu at (115.6, 158.8)
- added H5: MountingHole, MountingHole:MountingHole_6.4mm_M6, F.Cu at (63.2, 158.8)
- added H6: MountingHole, MountingHole:MountingHole_6.4mm_M6, F.Cu at (89.4, 158.8)
- added J3: Conn_01x03_Female, Connector_PinSocket_2.54mm:PinSocket_1x03_P2.54mm_Vertical, F.Cu at (78.6, 127.7)
- added J4: Conn_01x02_Female, TerminalBlock_Phoenix:TerminalBlock_Phoenix_MKDS-1,5-2_1x02_P5.00mm_Horizontal, F.Cu at (102.0, 85.9)
- added J6: USB_A, Connector_USB:USB_A_CONNFLY_DS1095-WNR0, F.Cu at (109.0, 130.9)
- added J7: Conn_01x11_Female, Connector_PinSocket_2.54mm:PinSocket_1x11_P2.54mm_Vertical, F.Cu at (41.7, 149.3)
- added R1: 75K, Resistor_THT:R_Axial_DIN0309_L9.0mm_D3.2mm_P12.70mm_Horizontal, F.Cu at (103.1, 120.3)
- added R2: 49.9K, Resistor_THT:R_Axial_DIN0309_L9.0mm_D3.2mm_P12.70mm_Horizontal, F.Cu at (98.5, 150.7)
- added R3: 75K, Resistor_THT:R_Axial_DIN0309_L9.0mm_D3.2mm_P12.70mm_Horizontal, F.Cu at (97.4, 120.2)
- added R4: 49.9K, Resistor_THT:R_Axial_DIN0309_L9.0mm_D3.2mm_P12.70mm_Horizontal, F.Cu at (98.4, 145.4)
- J1: value Conn_01x08_Female -> Conn_01x04_Female; footprint Connector_PinSocket_2.54mm:PinSocket_1x08_P2.54mm_Vertical -> Connector_PinSocket_2.54mm:PinSocket_1x04_P2.54mm_Vertical
- J2: value Screw_Terminal_01x02 -> Conn_01x02_Female; footprint TerminalBlock_Phoenix:TerminalBlock_Phoenix_MKDS-1,5-2-5.08_1x02_P5.08mm_Horizontal -> Connector_JST:JST_PH_S2B-PH-K_1x02_P2.00mm_Horizontal
- moved J1 94.9 mm to (77.9, 149.2), turned to 90 degrees
- moved J2 17.2 mm to (54.1, 88.2), turned to 180 degrees
Connections:
- J1 pad 1: 5V -> OUT
- J1 pad 3: (no net) -> 5VBOOST
- J1 pad 4: GND -> (no net)
- J2 pad 1: GND -> (no net)
- J2 pad 2: 5V -> (no net)
Routing:
- net (no net): vias 6 -> 0
Other:
- board size 100.9 x 90.4 mm -> 92.5 x 88.1 mm
- board text removed: "JST"
- board text removed: "USB"
- board text removed: "uUSB"

Commit message: boost_v1 sent to fab
Parts:
- moved R3 6.18 mm to (103.4, 121.7)
- moved R2 5.18 mm to (98.0, 145.5)
- moved R1 4.54 mm to (98.8, 121.7)
- moved R4 4.52 mm to (98.0, 149.9)
- moved C1 2.83 mm to (91.4, 127.8), turned to 270 degrees
- moved C2 2.59 mm to (91.4, 120.9), turned to 270 degrees
- moved J2 1.73 mm to (54.4, 89.9)
- moved J4 1.44 mm to (102.1, 87.4)
- moved D1 1.42 mm to (92.2, 136.7)
- moved F1 0.95 mm to (112.8, 141.5)
- moved J3 0.32 mm to (78.6, 128.0)
- renumbered H5 to H4, H6 to H5, H4 to H6
Connections:
- BT1 pad 1: (no net) -> LIPO
- BT1 pad 2: (no net) -> GND
- J2 pad 1: (no net) -> LIPO
- J2 pad 2: (no net) -> GND
- J7 pad 10: (no net) -> LIPO
Routing:
- net GND: track 0.00 -> 338.3 mm, vias 0 -> 5
- net LIPO: track 0.00 -> 138.1 mm, vias 0 -> 3
- net Net-(F1-Pad2): track 0.00 -> 75.3 mm
- net VUSB: track 0.00 -> 62.6 mm, vias 0 -> 1
- net 5VBOOST: track 0.00 -> 55.6 mm, vias 0 -> 5
- net Net-(C1-Pad1): track 0.00 -> 49.2 mm, vias 0 -> 2
- net Net-(C2-Pad1): track 0.00 -> 45.5 mm
- net Net-(J6-Pad2): track 0.00 -> 41.2 mm, vias 0 -> 2
- net Net-(J6-Pad3): track 0.00 -> 28.8 mm, vias 0 -> 1
- net OUT: track 0.00 -> 27.7 mm, vias 0 -> 2
Other:
- board text added: "+"
- board text added: "-"
- board text added: "5-10V IN"
- board text added: "5V"
- board text added: "5V USB OUT"
- board text added: "Adafruit Universal Lipo Charger"
- board text added: "GND"
- board text added: "LIPO"
- board text added: "TPS61023"
- board text added: "USBC"
- board text added: "VEXT"
- board text added: "VUSB"
- board text added: "pvos.org/power/boost_1"
- board text removed: "BOOSTA ver 0.1"
